Commit message: Added dae-model for C920 webcam; launch file to view model standalone

File: robotino_description/urdf/sensors/camera.urdf.xacro (robot description, xacro)
@@ -2,5 +2,5 @@
 <robot name="sensor_camera" xmlns:xacro="http://wiki.ros.org/xacro">
   <xacro:property name="M_PI" value="3.14159"/>
-  <xacro:property name="CAM_SCALE" value="0.01"/>
+  <xacro:property name="CAM_SCALE" value="1"/>
   <xacro:macro name="webcam" params="parent name *origin">
     <joint name="${name}_joint" type="fixed">
@@ -19,8 +19,8 @@
       <visual>
         <geometry>
-          <!--<mesh filename="package://robotino_description/meshes/sensors/c920.stl" scale="${CAM_SCALE} ${CAM_SCALE} ${CAM_SCALE}"/>-->
-		<box size="0.07 .09 .07"/>
+          <mesh filename="package://robotino_description/meshes/sensors/c920_small.dae" scale="${CAM_SCALE} ${CAM_SCALE} ${CAM_SCALE}"/>
+		<!--<box size="0.07 .09 .07"/>-->
         </geometry>
-		<origin rpy="0 0 0" xyz="0 0 0.035"/>
+		<origin rpy="0 0 0" xyz="-0.04 0 0.02"/>
       </visual>
     </link>
