Commit message: Reworked V3 model, separated base, pole and plates

File: robotino_description/urdf/robotino.urdf.xacro (robot description, xacro)
@@ -8,23 +8,45 @@
   <xacro:include filename="$(find robotino_description)/urdf/sensors/lzru901.urdf.xacro"/>
   <robotino_body/>
-  <!-- add platform -->
-    <platform name="platform" parent="base_link">
+  <!-- add pole -->
+    <pole name="pole" parent="base_link">
         <origin xyz="0.0 0.0 0.18" rpy="0 0 0"/>
+    </pole>
+  <!-- add 3 platforms as ring
+    <platform name="platform1" parent="pole_link">
+        <origin xyz="0.0288 0.0 0.19" rpy="0 0 0"/>
     </platform>
-  <!-- add kinect -->
-    <kinect name="camera" parent="base_link">
-        <origin xyz="0.1 0.0 0.68"/>
-    </kinect>
+    <platform name="platform2" parent="pole_link">
+        <origin xyz="-0.0144 0.0249 0.19" rpy="0 0 ${2*M_PI/3}"/>
+    </platform>
+    <platform name="platform3" parent="pole_link">
+        <origin xyz="-0.0144 -0.0249 0.19" rpy="0 0 ${4*M_PI/3}"/>
+    </platform>-->
+  <!-- add platform1-->
+    <platform name="platform1" parent="pole_link">
+        <origin xyz="0.0288 0.0 0.19" rpy="0 0 0"/>
+    </platform>
+  <!-- add platform2-->
+    <platform name="platform2" parent="pole_link">
+        <origin xyz="0.0288 0.0 0.39" rpy="0 0 0"/>
+    </platform>
+  <!-- add platform3-->
+    <platform name="platform3" parent="pole_link">
+        <origin xyz="0.0288 0.0 0.59" rpy="0 0 0"/>
+    </platform>
   <!-- add hokuyo -->
-    <hokuyo name="laser" parent="base_link">
-        <origin xyz="0.09 0.0 0.31"/>
+    <hokuyo name="laser" parent="pole_link">
+        <origin xyz="0.06 0.0 0.08"/>
     </hokuyo>
   <!-- add lzru901 -->
     <lzru901 name="laser_lzru901" parent="base_link">
-        <origin xyz="0.15 0.0 0.17"/>
+        <origin xyz="0.12 0.0 0.17"/>
     </lzru901>
   <!-- add webcam -->
-    <webcam name="webcam" parent="base_link">
-        <origin xyz="0.20 0.0 0.38"/>
+    <webcam name="webcam" parent="platform1_link">
+        <origin xyz="0.16 0.0 0.01"/>
     </webcam>
+  <!-- add kinect -->
+    <kinect name="camera" parent="platform2_link">
+        <origin xyz="0.07 0.0 0.08"/>
+    </kinect>
 </robot>

File: robotino_description/urdf/robotino_body.urdf.xacro (robot description, xacro)
@@ -2,5 +2,5 @@
 <robot xmlns:xacro="http://wiki.ros.org/xacro">
     <xacro:property name="M_PI" value="3.14159"/>
-    <xacro:property name="BASE_SCALE" value="0.001"/>
+    <xacro:property name="BASE_SCALE" value="1"/>
     <xacro:property name="BASE_RADIUS" value="0.23"/>
     <xacro:property name="BASE_HEIGHT" value="0.06"/>
@@ -18,7 +18,7 @@
             </inertial>
             <visual>
-                <origin xyz="0.01 0 0" rpy="0 0 ${M_PI}"/>
+                <origin xyz="0 0 0" rpy="0 0 0"/>
                 <geometry>
-                    <mesh filename="package://robotino_description/meshes/parts/robotino_v3.dae"
+                    <mesh filename="package://robotino_description/meshes/parts/robotino_v3_base.dae"
                         scale="${BASE_SCALE} ${BASE_SCALE} ${BASE_SCALE}"/>
                 </geometry>
@@ -52,7 +52,4 @@
             <origin xyz="-0.05 0 0.13" rpy="0 0 ${M_PI/2}"/>
         </command_bridge>-->
-        <!--<anglebracketusb name="anglebracketusb" parent="base_link">
-            <origin xyz="0.008 0 0.137" rpy="0 0 ${M_PI/2}"/>
-        </anglebracketusb>-->
         <!-- gazebo control -->
         <gazebo>

File: robotino_description/urdf/robotino_parts.urdf.xacro (robot description, xacro)
@@ -3,5 +3,6 @@
     <xacro:property name="M_PI" value="3.14159"/>
     <xacro:property name="M_SCALE" value="0.01"/>
-    <xacro:property name="PLATFORM_HEIGHT" value="0.59"/>
+    <xacro:property name="V3_SCALE" value="1"/>
+    <xacro:property name="POLE_HEIGHT" value="0.59"/>
     <xacro:property name="PLATFORM_RADIUS" value="0.225"/>
     <!-- wheel -->
@@ -60,6 +61,6 @@
         </joint>
     </xacro:macro>
-    <!-- angle bracket with USB hub -->
-    <xacro:macro name="anglebracketusb" params="parent name *origin">
+    <!-- pole -->
+    <xacro:macro name="pole" params="parent name *origin">
         <link name="${name}_link">
             <inertial>
@@ -69,9 +70,16 @@
             </inertial>
             <visual>
-                <origin xyz="0 0 0" rpy="0 0 0"/>
+                <origin xyz="0 0 0"/>
                 <geometry>
-                    <mesh filename="package://robotino_description/meshes/parts/angle_bracket_usb_hub.dae" scale="${M_SCALE} ${M_SCALE} ${M_SCALE}"/>
+                    <!--<cylinder radius="0.04" length="${POLE_HEIGHT}"/>-->
+			<mesh filename="package://robotino_description/meshes/parts/robotino_v3_pole.dae" scale="${V3_SCALE} ${V3_SCALE} ${V3_SCALE}"/>
                 </geometry>
             </visual>
+            <collision>
+                <origin xyz="0 0 ${POLE_HEIGHT/2}"/>
+                <geometry>
+                    <cylinder radius="0.04" length="${POLE_HEIGHT}"/>
+                </geometry>
+            </collision>
         </link>
         <joint name="${name}_joint" type="fixed">
@@ -90,14 +98,8 @@
             </inertial>
             <visual>
-                <origin xyz="0 0 ${PLATFORM_HEIGHT/2}"/>
+                <origin xyz="0 0 0"/>
                 <geometry>
-                    <cylinder radius="0.04" length="${PLATFORM_HEIGHT}"/>
-                </geometry>
-            </visual>
-            <visual>
-                <origin xyz="0 0 ${PLATFORM_HEIGHT}"/>
-                <geometry>
-                    <!-- actual length = 0.015 -->
-                    <cylinder radius="${PLATFORM_RADIUS}" length="0.02"/>
+                    <!--<cylinder radius="0.04" length="${POLE_HEIGHT}"/>-->
+			<mesh filename="package://robotino_description/meshes/parts/robotino_v3_plate.dae" scale="${V3_SCALE} ${V3_SCALE} ${V3_SCALE}"/>
                 </geometry>
             </visual>

File: robotino_description/urdf/sensors/lzru901.urdf.xacro (robot description, xacro)
@@ -22,8 +22,9 @@
         <origin xyz="0 0 -${LZR_LENGTH/4}" rpy="0 0 0" />
         <geometry>
-          <!--<mesh
-filename="package://robotino_description/meshes/sensors/hokuyo.dae" scale="${M_SCALE} ${M_SCALE} ${M_SCALE}"/>-->
-	<cylinder radius="${LZR_RADIUS}" length="${LZR_LENGTH}" />
+	  <cylinder radius="${LZR_RADIUS}" length="${LZR_LENGTH}" />
         </geometry>
+	<material name="black">
+          <color rgba="0 0 0 1"/>
+      	</material>
       </visual>
       <collision>

Commit message: Integrated Kinect V2 model and cleanup

File: robotino_description/urdf/robotino.urdf.xacro (robot description, xacro)
@@ -7,4 +7,5 @@
   <xacro:include filename="$(find robotino_description)/urdf/sensors/camera.urdf.xacro"/>
   <xacro:include filename="$(find robotino_description)/urdf/sensors/lzru901.urdf.xacro"/>
+  <xacro:include filename="$(find robotino_description)/urdf/sensors/kinectv2.urdf.xacro"/>
   <robotino_body/>
   <!-- add pole -->
@@ -50,3 +51,7 @@
         <origin xyz="0.07 0.0 0.08"/>
     </kinect>
+  <!-- add kinect v2 -->
+    <kinectv2 name="kinectv2" parent="platform3_link">
+        <origin xyz="0.07 0.0 0.04"/>
+    </kinectv2>
 </robot>
