Commit message: minor changes

File: robotino_description3/urdf/robotino300252.urdf.xacro (robot description, xacro)
@@ -37,9 +37,9 @@
   <!-- add hokuyo -->
     <hokuyo name="laser" parent="platform1_link">
-        <origin xyz="0.11 0.0 0.06"/>
+        <origin xyz="0.11 0.0 0.0"/>
     </hokuyo>
   <!-- add webcam -->
     <webcam name="webcam" parent="pole_link">
-        <origin xyz="0.01 0.0 0.35"/>
+        <origin xyz="0.07 0.0 0.35"/>
     </webcam>
   <!-- add kinect -->

Commit message: change in urdf

File: robotino_description3/urdf/robotino300252.urdf.xacro (robot description, xacro)
@@ -45,5 +45,5 @@
   <!-- add kinect -->
     <kinect name="camera" parent="platform2_link">
-        <origin xyz="0.10 0.0 0.08"/>
+        <origin xyz="0.10 0.0 0.0"/>
     </kinect>
   <!-- add kinect v2

Commit message: Changed Robotino 252 URDF

File: robotino_description3/urdf/robotino300252.urdf.xacro (robot description, xacro)
@@ -23,8 +23,8 @@
         <origin xyz="-0.0144 -0.0249 0.19" rpy="0 0 ${4*M_PI/3}"/>
     </platform>-->
-  <!-- add platform1-->
+  <!-- add platform1
     <platform name="platform1" parent="pole_link">
         <origin xyz="0.0288 0.0 0.18" rpy="0 0 0"/>
-    </platform>
+    </platform>-->
   <!-- add platform2-->
     <platform name="platform2" parent="pole_link">
@@ -36,6 +36,6 @@
     </platform>-->
   <!-- add hokuyo -->
-    <hokuyo name="laser" parent="platform1_link">
-        <origin xyz="0.11 0.0 0.0"/>
+    <hokuyo name="laser" parent="pole_link">
+        <origin xyz="0.07 0.0 0.12"/>
     </hokuyo>
   <!-- add webcam -->

Commit message: Small error in URDF of Robot 252

File: robotino_description3/urdf/robotino300252.urdf.xacro (robot description, xacro)
@@ -45,5 +45,5 @@
   <!-- add kinect -->
     <kinect name="camera" parent="platform2_link">
-        <origin xyz="0.10 0.0 0.0"/>
+        <origin xyz="0.10 0.0 0.05"/>
     </kinect>
   <!-- add kinect v2
